File: P00_ThreadControl/C02_DisplayControl/P00_C02_H00_DisplayControl/P00_C02_H00_DisplayControl.kicad_pcb (KiCad board)
At the start: 2 copper layers, 100 x 14 mm, 73 parts, among them IC1 AP2139AK-3.3, IC2 STM32F030F4P6, IC3 FT230XS, IC4 VEML6030, IC5 VL53L0X, Q1 ECS-160-8-30Q-VY, T1 BC847B,215, T2 BC847B,215, T3 BC847B,215, X1 FTSH-105-01-F-DV-K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

Commit message: Final PCB Version 1.0. These files where send to the manufacturer.
Parts:
- moved LED1 11.3 mm to (116.9, 87.0)
- moved LED2 8.05 mm to (115.3, 87.0)
- moved FB3 6.73 mm to (117.0, 86.5), turned to 90 degrees
- moved C9 6.72 mm to (116.1, 86.4), turned to 270 degrees
- moved FB2 5.82 mm to (143.9, 90.4), turned to 180 degrees
- moved FB4 5.68 mm to (132.0, 89.0)
- moved FB7 5.57 mm to (134.5, 88.4), turned to 270 degrees
- moved C24 5.34 mm to (133.2, 86.8), turned to 90 degrees
- moved R22 5.28 mm to (129.5, 91.7)
- moved C19 5.01 mm to (119.2, 85.5)
- moved C2 5.00 mm to (157.6, 82.8)
- moved C16 5.00 mm to (119.2, 83.2)
- moved Q1 5.00 mm to (121.5, 84.3)
- moved C3 5.00 mm to (152.6, 82.9)
- moved C17 5.00 mm to (129.8, 82.4)
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Connections:
- IC2 pad 11: /GPI_VEML6030_INT -> Net-(IC2-Pad11)
- IC2 pad 14: Net-(IC2-Pad14) -> /GPI_VEML6030_INT
- X2 pad M1: (no net) -> GND
- X2 pad M2: (no net) -> GND
- X2 pad M3: (no net) -> GND
- X2 pad M4: (no net) -> GND
- X2 pad M5: (no net) -> GND
- X2 pad M6: (no net) -> GND
Routing:
- net +5V: track 35.5 -> 23.2 mm, vias 2 -> 6
- net Net-(LED1-Pad2): track 11.3 -> 4.41 mm
- net +3V3: track 19.1 -> 12.7 mm, vias 5 -> 6
- net /SDA: track 42.2 -> 36.2 mm
- net /SCL: track 43.5 -> 37.6 mm
- net /GPI_VEML6030_INT: track 10.1 -> 6.84 mm
- net Net-(C13-Pad1): track 20.1 -> 23.3 mm
- net Net-(C1-Pad1): track 6.58 -> 4.69 mm
- net GND: track 83.5 -> 81.7 mm, vias 53 -> 142
- net /nRST: track 18.4 -> 20.1 mm
- net /GPI_VL53L0X_INT: track 34.8 -> 36.4 mm
- net Net-(C4-Pad1): track 6.95 -> 8.17 mm
- net Net-(C19-Pad1): track 6.97 -> 7.92 mm
- net Net-(C16-Pad1): track 8.37 -> 9.25 mm
- net Net-(C9-Pad1): track 4.70 -> 3.86 mm
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- added copper zone on B.Cu, net +5V
- added copper zone on F.Cu, net +5V
- added copper zone on B.Cu, net Net-(C1-Pad1)
Other:
- board size 100 x 14 mm -> 90 x 14 mm
