File: P00_ThreadControl/C02_DisplayControl/P00_C02_H00_DisplayControl/P00_C02_H00_DisplayControl.sch (KiCad schematic (older format))
At the start: 73 parts, among them IC1 AP2139AK-3.3, IC2 STM32F030F4P6, IC3 FT230XS, IC4 VEML6030, IC5 VL53L0X, Q1 ECS-160-8-30Q-VY, T1 BC847B,215, T2 BC847B,215, T3 BC847B,215, X1 FTSH-105-01-F-DV-K, X2 629105150921

Commit message: Final PCB Version 1.0. These files where send to the manufacturer.
Connections:
- net GPI_VEML6030_INT: now also IC2.14 (PB1); no longer IC2.11 (PA5)
Other:
- moved on the sheet: R20
Changed lines of the file:
@@
 Sheet 1 1
 Title "P00_C02_H00_DisplayControl"
-Date "2020-04-14"
+Date "2020-04-17"
 Rev "v1.0"
 Comp "Projektarbeit SS2020"
@@
 L resistor:RC0402FR-0710KL R20
 U 1 1 5E99B980
-P 9700 4350
-F 0 "R20" H 9700 4420 50  0000 C CNN
-F 1 "RC0402FR-0710KL" H 9700 4200 39  0001 C CNN
-F 2 "resistor:R0402" H 9700 4350 50  0001 C CNN
-F 3 "" H 9700 4350 50  0001 C CNN
-F 4 "0402" H 9700 4350 39  0000 C CNN "Package"
-F 5 "10k" H 9700 4275 50  0000 C CNN "Resistance"
-F 6 "Yageo" H 9700 4150 50  0001 C CNN "MFR"
-	1    9700 4350
-	1    0    0    -1
-$EndComp
-Text Label 9550 4200 0    50   ~ 0
+P 9400 5150
+F 0 "R20" H 9400 5220 50  0000 C CNN
+F 1 "RC0402FR-0710KL" H 9400 5000 39  0001 C CNN
+F 2 "resistor:R0402" H 9400 5150 50  0001 C CNN
+F 3 "" H 9400 5150 50  0001 C CNN
+F 4 "0402" H 9400 5150 39  0000 C CNN "Package"
+F 5 "10k" H 9400 5075 50  0000 C CNN "Resistance"
+F 6 "Yageo" H 9400 4950 50  0001 C CNN "MFR"
+	1    9400 5150
+	1    0    0    -1
+$EndComp
+Text Label 9250 5000 0    50   ~ 0
 GPI_VEML6030_INT
 Text Label 9550 4600 0    50   ~ 0
@@
 L power:GND #PWR038
 U 1 1 5E9A5634
-P 9900 4350
-F 0 "#PWR038" H 9900 4100 50  0001 C CNN
-F 1 "GND" H 9900 4200 50  0000 C CNN
-F 2 "" H 9900 4350 50  0001 C CNN
-F 3 "" H 9900 4350 50  0001 C CNN
-	1    9900 4350
+P 9600 5150
+F 0 "#PWR038" H 9600 4900 50  0001 C CNN
+F 1 "GND" H 9600 5000 50  0000 C CNN
+F 2 "" H 9600 5150 50  0001 C CNN
+F 3 "" H 9600 5150 50  0001 C CNN
+	1    9600 5150
 	0    -1   -1   0
 $EndComp
 Wire Wire Line
-	9900 4350 9850 4350
-Wire Wire Line
-	9550 4350 9500 4350
-Wire Wire Line
-	9500 4350 9500 4200
-Wire Wire Line
-	9500 4200 9550 4200
-Wire Wire Line
-	9500 4200 9500 3650
-Connection ~ 9500 4200
+	9600 5150 9550 5150
+Wire Wire Line
+	9250 5150 9200 5150
+Wire Wire Line
+	9200 5150 9200 5000
+Wire Wire Line
+	9200 5000 9250 5000
+Wire Wire Line
+	9200 5000 9200 4450
+Connection ~ 9200 5000
 $Comp
 L resistor:RC0402FR-0710KL R22
@@
 Wire Wire Line
 	9900 4750 9850 4750
-Wire Wire Line
-	9500 3650 8800 3650
 Wire Wire Line
 	9550 4750 9400 4750
@@
 Wire Wire Line
 	5800 5050 5800 5100
-NoConn ~ 8800 4450
 NoConn ~ 8800 3850
 Text Label 2050 6500 2    50   ~ 0
@@
 	1    0    0    -1
 $EndComp
+Wire Wire Line
+	8800 4450 9200 4450
+NoConn ~ 8800 3650
 $EndSCHEMATC

Commit message: Added manufacturer to capacitor fields in the lib.
Parts:
- C1, C10, C11, C12, C13, C14, C15, C16, C17, C18, C19, C2, C20, C21, C22, C23, C24, C25, C26, C27, C3, C4, C5, C6, C8, C9: MFR (none) -> Samsung Electro Mechanics
Changed lines of the file:
@@
 F 6 "0805" V 1490 3480 31  0000 L BNN "Package"
 F 7 "10u" H 1510 3410 50  0000 L TNN "Capacitance"
+F 8 "Samsung Electro Mechanics" H 0   0   50  0001 C CNN "MFR"
 	1    1500 3450
 	1    0    0    -1
@@
 F 6 "0805" V 1790 1230 31  0000 L BNN "Package"
 F 7 "10u" H 1810 1160 50  0000 L TNN "Capacitance"
+F 8 "Samsung Electro Mechanics" H 0   0   50  0001 C CNN "MFR"
 	1    1800 1200
 	1    0    0    -1
@@
 F 6 "0402" V 2040 1230 31  0000 L BNN "Package"
 F 7 "100n" H 2060 1160 50  0000 L TNN "Capacitance"
+F 8 "Samsung Electro Mechanics" H 0   0   50  0001 C CNN "MFR"
 	1    2050 1200
 	1    0    0    -1
@@
 F 6 "0402" V 2790 1230 31  0000 L BNN "Package"
 F 7 "100n" H 2810 1160 50  0000 L TNN "Capacitance"
+F 8 "Samsung Electro Mechanics" H 0   0   50  0001 C CNN "MFR"
 	1    2800 1200
 	1    0    0    -1
@@
 F 6 "0402" V 1740 3480 31  0000 L BNN "Package"
 F 7 "100n" H 1760 3410 50  0000 L TNN "Capacitance"
+F 8 "Samsung Electro Mechanics" H 0   0   50  0001 C CNN "MFR"
 	1    1750 3450
 	1    0    0    -1
@@
 F 6 "0402" V 2040 3580 31  0000 L BNN "Package"
 F 7 "100n" H 2060 3510 50  0000 L TNN "Capacitance"
+F 8 "Samsung Electro Mechanics" H 0   0   50  0001 C CNN "MFR"
 	1    2050 3550
 	1    0    0    -1
@@
 F 6 "0402" V 4140 4180 31  0000 L BNN "Package"
 F 7 "33p" H 4160 4110 50  0000 L TNN "Capacitance"
+F 8 "Samsung Electro Mechanics" H 0   0   50  0001 C CNN "MFR"
 	1    4150 4150
 	1    0    0    -1
@@
 F 6 "0402" V 4390 4180 31  0000 L BNN "Package"
 F 7 "33p" H 4410 4110 50  0000 L TNN "Capacitance"
+F 8 "Samsung Electro Mechanics" H 0   0   50  0001 C CNN "MFR"
 	1    4400 4150
 	1    0    0    -1
@@
 F 6 "0402" V 3890 1230 31  0000 L BNN "Package"
 F 7 "100n" H 3910 1160 50  0000 L TNN "Capacitance"
+F 8 "Samsung Electro Mechanics" H 0   0   50  0001 C CNN "MFR"
 	1    3900 1200
 	1    0    0    -1
@@
 F 6 "0805" V 3640 1230 31  0000 L BNN "Package"
 F 7 "10u" H 3660 1160 50  0000 L TNN "Capacitance"
+F 8 "Samsung Electro Mechanics" H 0   0   50  0001 C CNN "MFR"
 	1    3650 1200
 	1    0    0    -1
@@
 F 6 "0402" V 5040 1230 31  0000 L BNN "Package"
 F 7 "100n" H 5060 1160 50  0000 L TNN "Capacitance"
+F 8 "Samsung Electro Mechanics" H 0   0   50  0001 C CNN "MFR"
 	1    5050 1200
 	1    0    0    -1
@@
 F 6 "0402" V 10440 1330 31  0000 L BNN "Package"
 F 7 "100n" H 10460 1260 50  0000 L TNN "Capacitance"
+F 8 "Samsung Electro Mechanics" H 0   0   50  0001 C CNN "MFR"
 	1    10450 1300
 	1    0    0    -1
@@
 F 6 "0402" V 6540 3680 31  0000 L BNN "Package"
 F 7 "100n" H 6560 3610 50  0000 L TNN "Capacitance"
+F 8 "Samsung Electro Mechanics" H 0   0   50  0001 C CNN "MFR"
 	1    6550 3650
 	1    0    0    -1
@@
 F 6 "0402" V 6240 3680 31  0000 L BNN "Package"
 F 7 "100n" H 6260 3610 50  0000 L TNN "Capacitance"
+F 8 "Samsung Electro Mechanics" H 0   0   50  0001 C CNN "MFR"
 	1    6250 3650
 	1    0    0    -1
@@
 F 6 "0805" V 5940 3680 31  0000 L BNN "Package"
 F 7 "10u" H 5960 3610 50  0000 L TNN "Capacitance"
+F 8 "Samsung Electro Mechanics" H 0   0   50  0001 C CNN "MFR"
 	1    5950 3650
 	1    0    0    -1
@@
 F 6 "0402" V 7100 3920 31  0000 R BNN "Package"
 F 7 "12p" V 7160 3980 50  0000 L TNN "Capacitance"
+F 8 "Samsung Electro Mechanics" H 0   0   50  0001 C CNN "MFR"
 	1    7150 3950
 	0    1    1    0
@@
 F 6 "0402" V 7100 3620 31  0000 R BNN "Package"
 F 7 "12p" V 7160 3680 50  0000 L TNN "Capacitance"
+F 8 "Samsung Electro Mechanics" H 0   0   50  0001 C CNN "MFR"
 	1    7150 3650
 	0    1    1    0
@@
 F 6 "0402" V 6590 1830 31  0000 L BNN "Package"
 F 7 "100n" H 6610 1760 50  0000 L TNN "Capacitance"
+F 8 "Samsung Electro Mechanics" H 0   0   50  0001 C CNN "MFR"
 	1    6600 1800
 	1    0    0    -1
@@
 F 6 "0402" V 9640 3680 31  0000 L BNN "Package"
 F 7 "33p" H 9660 3610 50  0000 L TNN "Capacitance"
+F 8 "Samsung Electro Mechanics" H 0   0   50  0001 C CNN "MFR"
 	1    9650 3650
 	1    0    0    -1
@@
 F 6 "0402" V 9890 3680 31  0000 L BNN "Package"
 F 7 "33p" H 9910 3610 50  0000 L TNN "Capacitance"
+F 8 "Samsung Electro Mechanics" H 0   0   50  0001 C CNN "MFR"
 	1    9900 3650
 	1    0    0    -1
@@
 F 6 "0805" V 3940 6380 31  0000 L BNN "Package"
 F 7 "10u" H 3960 6310 50  0000 L TNN "Capacitance"
+F 8 "Samsung Electro Mechanics" H 0   0   50  0001 C CNN "MFR"
 	1    3950 6350
 	1    0    0    -1
@@
 F 6 "0402" V 3640 6380 31  0000 L BNN "Package"
 F 7 "100n" H 3660 6310 50  0000 L TNN "Capacitance"
+F 8 "Samsung Electro Mechanics" H 0   0   50  0001 C CNN "MFR"
 	1    3650 6350
 	1    0    0    -1
@@
 F 6 "0402" V 3340 6380 31  0000 L BNN "Package"
 F 7 "100n" H 3360 6310 50  0000 L TNN "Capacitance"
+F 8 "Samsung Electro Mechanics" H 0   0   50  0001 C CNN "MFR"
 	1    3350 6350
 	1    0    0    -1
@@
 F 6 "0805" V 6540 6230 31  0000 L BNN "Package"
 F 7 "10u" H 6560 6160 50  0000 L TNN "Capacitance"
+F 8 "Samsung Electro Mechanics" H 0   0   50  0001 C CNN "MFR"
 	1    6550 6200
 	1    0    0    -1
@@
 F 6 "0402" V 6240 6230 31  0000 L BNN "Package"
 F 7 "100n" H 6260 6160 50  0000 L TNN "Capacitance"
+F 8 "Samsung Electro Mechanics" H 0   0   50  0001 C CNN "MFR"
 	1    6250 6200
 	1    0    0    -1
@@
 F 6 "0402" V 1140 6530 31  0000 L BNN "Package"
 F 7 "100n" H 1160 6460 50  0000 L TNN "Capacitance"
+F 8 "Samsung Electro Mechanics" H 0   0   50  0001 C CNN "MFR"
 	1    1150 6500
 	1    0    0    -1
